File: city.kicad_sch (KiCad schematic)
At the start: 28 parts, among them J1 USB_C_Receptacle_USB2.0_16P, J4 Conn_01x08_Pin, J5 Conn_01x08_Pin, SW1 SW_Push, SW2 SW_Push, U1 USBLC6-2SC6, U2 AP2112K-3.3, U3 ESP32-C3-WROOM-02, Y1 Crystal

Commit message: starting to add fixes and changing some dimensions
Parts:
- added J2: Conn_01x04, Connector_PinHeader_2.00mm:PinHeader_1x04_P2.00mm_Vertical, symbol Connector_Generic:Conn_01x04
Connections:
- net +3.3V: now also J2.1 (Pin_1)
- net GND: now also J2.4 (Pin_4)
- net RXD: now also J2.3 (Pin_3)
- net TXD: now also J2.2 (Pin_2)
